File: noise-a-tron.kicad_pcb (KiCad board)
At the start: 2 copper layers, 100 x 62.3 mm, 27 parts, among them Q1 BC557, Q2 MMBT3906, SW1 SW_Push, SW2 SW_Push, SW3 SW_Push, SW4 SW_Push, SW5 SW_Push, SW6 SW_Push, SW7 SW_Push, U1 74HC00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

Commit message: Added JLCJLCJLCJLC
Other:
- board text added: "JLCJLCJLCJLC"
Changed lines of the file:
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@@
     (effects (font (size 1 1) (thickness 0.15)) (justify left bottom mirror))
+  )
+  (gr_text "JLCJLCJLCJLC" (at 102.35 111.25) (layer "F.SilkS")
+    (effects (font (size 0.9 0.9) (thickness 0.15)) (justify left bottom))
   )
   (segment (start 187.5 124.6) (end 187.75 124.35) (width 1) (layer "F.Cu") (net 1))
